File: electronics/control/control.sch (KiCad schematic (older format))
At the start: 20 parts

Commit message: Add the PCB.
Parts:
- C1: renamed from C?; footprint (none) -> Capacitor_SMD:C_0805_2012Metric
- C2: renamed from C?; value 1µF/10V -> 1µF/20V; footprint (none) -> Capacitor_SMD:C_0805_2012Metric
- C3, C9: renamed from C?; value 1000µF/10V -> 1000µF/20V; footprint (none) -> Capacitor_THT:CP_Radial_D10.0mm_P5.00mm
- C4, C6: renamed from C?; value 18pF/10V -> 18pF/20V; footprint (none) -> Capacitor_SMD:C_0805_2012Metric
- C5: renamed from C?; value 0.1µF/10V Low ESR -> 0.1µF/20V; footprint (none) -> Capacitor_SMD:C_0805_2012Metric
- C7: renamed from C?; value 2.2µF/10V -> 2.2µF/20V; footprint (none) -> Capacitor_SMD:C_0805_2012Metric
- C8: renamed from C?; value 10µF/10V Low ESR -> 10µF/20V; footprint (none) -> Capacitor_SMD:C_0805_2012Metric
- D1, D2: renamed from D?; value D -> S1B-13-F; footprint (none) -> Diode_SMD:D_SMA
- J1: renamed from J?; footprint (none) -> CNC:EBWA-02-B
- J2: renamed from J?; footprint (none) -> Connector_USB:USB_B_OST_USB-B1HSxx_Horizontal
- JP1: renamed from JP?; footprint (none) -> Connector_PinHeader_2.54mm:PinHeader_1x03_P2.54mm_Vertical
- R1, R2: renamed from R?; footprint (none) -> Resistor_SMD:R_0805_2012Metric
- RV1: renamed from RV?; footprint (none) -> Resistor_SMD:R_0805_2012Metric
- U1: renamed from U?; footprint (none) -> Package_TO_SOT_SMD:SOT-23-6
- U10: renamed from U?; footprint (none) -> Package_TO_SOT_SMD:SOT-89-3
- U11: renamed from U?; footprint (none) -> Package_TO_SOT_SMD:SOT-223-3_TabPin2
Connections:
- net J2_D-: now reaches J2.2 (D-), R2.1, U1.1 (I/O)
- net J2_D+: now reaches J2.3 (D+), R1.1, U1.6 (I/O)
Changed lines of the file:
@@
 P 3050 6800
 AR Path="/606CB5C7/60B0C177" Ref="U?"  Part="1"
-AR Path="/60B0C177" Ref="U?"  Part="1"
-F 0 "U?" H 3100 6915 50  0000 C CNN
+AR Path="/60B0C177" Ref="U10"  Part="1"
+F 0 "U10" H 3100 6915 50  0000 C CNN
 F 1 "AP7381_SOT89" H 3100 6824 50  0000 C CNN
-F 2 "" H 3050 6800 50  0001 C CNN
+F 2 "Package_TO_SOT_SMD:SOT-89-3" H 3050 6800 50  0001 C CNN
 F 3 "" H 3050 6800 50  0001 C CNN
 	1    3050 6800
@@
 P 2300 7200
 AR Path="/606CB5C7/60B0C18B" Ref="C?"  Part="1"
-AR Path="/60B0C18B" Ref="C?"  Part="1"
-F 0 "C?" H 2415 7246 50  0000 L CNN
-F 1 "1µF/10V" H 2415 7155 50  0000 L CNN
-F 2 "" H 2338 7050 50  0001 C CNN
+AR Path="/60B0C18B" Ref="C2"  Part="1"
+F 0 "C2" H 2415 7246 50  0000 L CNN
+F 1 "1µF/20V" H 2415 7155 50  0000 L CNN
+F 2 "Capacitor_SMD:C_0805_2012Metric" H 2338 7050 50  0001 C CNN
 F 3 "~" H 2300 7200 50  0001 C CNN
 	1    2300 7200
@@
 P 3700 7200
 AR Path="/606CB5C7/60B0C191" Ref="C?"  Part="1"
-AR Path="/60B0C191" Ref="C?"  Part="1"
-F 0 "C?" H 3815 7246 50  0000 L CNN
-F 1 "2.2µF/10V" H 3815 7155 50  0000 L CNN
-F 2 "" H 3738 7050 50  0001 C CNN
+AR Path="/60B0C191" Ref="C7"  Part="1"
+F 0 "C7" H 3815 7246 50  0000 L CNN
+F 1 "2.2µF/20V" H 3815 7155 50  0000 L CNN
+F 2 "Capacitor_SMD:C_0805_2012Metric" H 3738 7050 50  0001 C CNN
 F 3 "~" H 3700 7200 50  0001 C CNN
 	1    3700 7200
@@
 ENDSTOPS_3.3V
 $Comp
-L Jumper:Jumper_3_Open JP?
+L Jumper:Jumper_3_Open JP1
 U 1 1 606EA413
 P 1150 5200
-F 0 "JP?" V 1196 5287 50  0000 L CNN
+F 0 "JP1" V 1196 5287 50  0000 L CNN
 F 1 "5V" V 1105 5287 50  0000 L CNN
-F 2 "" H 1150 5200 50  0001 C CNN
+F 2 "Connector_PinHeader_2.54mm:PinHeader_1x03_P2.54mm_Vertical" H 1150 5200 50  0001 C CNN
 F 3 "~" H 1150 5200 50  0001 C CNN
 	1    1150 5200
@@
 $EndComp
 $Comp
-L Connector:Conn_01x02_Female J?
+L Connector:Conn_01x02_Female J1
 U 1 1 606EC204
 P 850 4750
-F 0 "J?" H 742 4935 50  0000 C CNN
+F 0 "J1" H 742 4935 50  0000 C CNN
 F 1 "5V" H 742 4844 50  0000 C CNN
-F 2 "" H 850 4750 50  0001 C CNN
+F 2 "CNC:EBWA-02-B" H 850 4750 50  0001 C CNN
 F 3 "~" H 850 4750 50  0001 C CNN
 	1    850  4750
@@
 	1050 4750 1600 4750
 $Comp
-L CNC:LM2937IMP-3.3 U?
+L CNC:LM2937IMP-3.3 U11
 U 1 1 606F2EC9
 P 4750 5050
-F 0 "U?" H 4800 5165 50  0000 C CNN
+F 0 "U11" H 4800 5165 50  0000 C CNN
 F 1 "LM2937IMP-3.3" H 4800 5074 50  0000 C CNN
-F 2 "" H 4750 5050 50  0001 C CNN
+F 2 "Package_TO_SOT_SMD:SOT-223-3_TabPin2" H 4750 5050 50  0001 C CNN
 F 3 "" H 4750 5050 50  0001 C CNN
 	1    4750 5050
@@
 Connection ~ 2900 5200
 $Comp
-L Device:C C?
+L Device:C C5
 U 1 1 606F487D
 P 3400 5450
-F 0 "C?" H 3515 5496 50  0000 L CNN
-F 1 "0.1µF/10V Low ESR" H 3515 5405 50  0000 L CNN
-F 2 "" H 3438 5300 50  0001 C CNN
+F 0 "C5" H 3515 5496 50  0000 L CNN
+F 1 "0.1µF/20V" H 3515 5405 50  0000 L CNN
+F 2 "Capacitor_SMD:C_0805_2012Metric" H 3438 5300 50  0001 C CNN
 F 3 "~" H 3400 5450 50  0001 C CNN
 	1    3400 5450
@@
 	3400 5700 3400 5600
 $Comp
-L Device:C C?
+L Device:C C8
 U 1 1 606F9DA2
 P 5300 5450
-F 0 "C?" H 5415 5496 50  0000 L CNN
-F 1 "10µF/10V Low ESR" H 5415 5405 50  0000 L CNN
-F 2 "" H 5338 5300 50  0001 C CNN
+F 0 "C8" H 5415 5496 50  0000 L CNN
+F 1 "10µF/20V" H 5415 5405 50  0000 L CNN
+F 2 "Capacitor_SMD:C_0805_2012Metric" H 5338 5300 50  0001 C CNN
 F 3 "~" H 5300 5450 50  0001 C CNN
 	1    5300 5450
@@
 	5300 5200 5200 5200
 $Comp
-L Device:CP C?
+L Device:CP C3
 U 1 1 6070A91B
 P 2500 5450
-F 0 "C?" H 2618 5496 50  0000 L CNN
-F 1 "1000µF/10V" H 2618 5405 50  0000 L CNN
-F 2 "" H 2538 5300 50  0001 C CNN
+F 0 "C3" H 2618 5496 50  0000 L CNN
+F 1 "1000µF/20V" H 2618 5405 50  0000 L CNN
+F 2 "Capacitor_THT:CP_Radial_D10.0mm_P5.00mm" H 2538 5300 50  0001 C CNN
 F 3 "~" H 2500 5450 50  0001 C CNN
 	1    2500 5450
@@
 	2500 5700 2500 5600
 $Comp
-L Device:CP C?
+L Device:CP C9
 U 1 1 607123DE
 P 6300 5450
-F 0 "C?" H 6418 5496 50  0000 L CNN
-F 1 "1000µF/10V" H 6418 5405 50  0000 L CNN
-F 2 "" H 6338 5300 50  0001 C CNN
+F 0 "C9" H 6418 5496 50  0000 L CNN
+F 1 "1000µF/20V" H 6418 5405 50  0000 L CNN
+F 2 "Capacitor_THT:CP_Radial_D10.0mm_P5.00mm" H 6338 5300 50  0001 C CNN
 F 3 "~" H 6300 5450 50  0001 C CNN
 	1    6300 5450
@@
 	6300 5700 6300 5600
 $Comp
-L Connector:USB_B J?
+L Connector:USB_B J2
 U 1 1 607151A5
 P 1000 1500
-F 0 "J?" H 1057 1967 50  0000 C CNN
+F 0 "J2" H 1057 1967 50  0000 C CNN
 F 1 "USB_B" H 1057 1876 50  0000 C CNN
-F 2 "" H 1150 1450 50  0001 C CNN
+F 2 "Connector_USB:USB_B_OST_USB-B1HSxx_Horizontal" H 1150 1450 50  0001 C CNN
 F 3 " ~" H 1150 1450 50  0001 C CNN
 	1    1000 1500
@@
 Wire Wire Line
 	1150 5600 1150 5450
-$Comp
-L CNC:NUP2114UCMR6T1G U?
-U 1 1 607223C1
-P 2100 1600
-F 0 "U?" H 2000 1000 50  0000 C CNN
-F 1 "NUP2114UCMR6T1G" H 2000 900 50  0000 C CNN
-F 2 "" H 2100 1600 50  0001 C CNN
-F 3 "" H 2100 1600 50  0001 C CNN
-	1    2100 1600
-	1    0    0    -1
-$EndComp
 $Comp
 L power:GNDD #PWR?
@@
 $EndComp
 $Comp
-L Device:Varistor RV?
+L Device:Varistor RV1
 U 1 1 6073FBA4
 P 1500 5600
-F 0 "RV?" H 1603 5646 50  0000 L CNN
+F 0 "RV1" H 1603 5646 50  0000 L CNN
 F 1 "B72510T0040M062" H 1603 5555 50  0000 L CNN
-F 2 "" V 1430 5600 50  0001 C CNN
+F 2 "Resistor_SMD:R_0805_2012Metric" V 1430 5600 50  0001 C CNN
 F 3 "~" H 1500 5600 50  0001 C CNN
 	1    1500 5600
@@
 $EndComp
 $Comp
-L Device:C C?
+L Device:C C1
 U 1 1 60740843
 P 900 2450
-F 0 "C?" H 1015 2496 50  0000 L CNN
+F 0 "C1" H 1015 2496 50  0000 L CNN
 F 1 "4700pF" H 1015 2405 50  0000 L CNN
-F 2 "" H 938 2300 50  0001 C CNN
+F 2 "Capacitor_SMD:C_0805_2012Metric" H 938 2300 50  0001 C CNN
 F 3 "~" H 900 2450 50  0001 C CNN
 	1    900  2450
@@
 Connection ~ 2400 1500
 $Comp
-L Device:R R?
+L Device:R R1
 U 1 1 60782E21
 P 3050 1400
-F 0 "R?" V 3257 1400 50  0000 C CNN
+F 0 "R1" V 3257 1400 50  0000 C CNN
 F 1 "33" V 3166 1400 50  0000 C CNN
-F 2 "" V 2980 1400 50  0001 C CNN
+F 2 "Resistor_SMD:R_0805_2012Metric" V 2980 1400 50  0001 C CNN
 F 3 "~" H 3050 1400 50  0001 C CNN
 	1    3050 1400
@@
 $EndComp
 $Comp
-L Device:R R?
+L Device:R R2
 U 1 1 60783483
 P 3050 1700
-F 0 "R?" V 3257 1700 50  0000 C CNN
+F 0 "R2" V 3257 1700 50  0000 C CNN
 F 1 "33" V 3166 1700 50  0000 C CNN
-F 2 "" V 2980 1700 50  0001 C CNN
+F 2 "Resistor_SMD:R_0805_2012Metric" V 2980 1700 50  0001 C CNN
 F 3 "~" H 3050 1700 50  0001 C CNN
 	1    3050 1700
@@
 F11 "X_DIR" O R 5750 1950 50
 F12 "X_STEP" O R 5750 2050 50
-F13 "Y_DIR" O R 5750 2200 50
-F14 "Y_STEP" O R 5750 2300 50
-F15 "Z_EN" O R 5750 2400 50
-F16 "Z_DIR" O R 5750 2550 50
-F17 "Z_STEP" O R 5750 2650 50
-F18 "Y_EN" O R 5750 2750 50
-F19 "SPINDLE_FEEDBACK" I R 5750 3250 50
-F20 "SPINDLE_PWM" O R 5750 3350 50
+F13 "Y_DIR" O R 5750 2300 50
+F14 "Y_STEP" O R 5750 2400 50
+F15 "Z_EN" O R 5750 2550 50
+F16 "Z_DIR" O R 5750 2650 50
+F17 "Z_STEP" O R 5750 2750 50
+F18 "Y_EN" O R 5750 2200 50
+F19 "SPINDLE_FEEDBACK" I R 5750 3350 50
+F20 "SPINDLE_PWM" O R 5750 3250 50
 $EndSheet
 $Comp
@@
 Voltage regulators
 $Comp
-L Device:D D?
+L Device:D D1
 U 1 1 607D55EE
 P 3100 6450
-F 0 "D?" H 3100 6667 50  0000 C CNN
-F 1 "D" H 3100 6576 50  0000 C CNN
-F 2 "" H 3100 6450 50  0001 C CNN
+F 0 "D1" H 3100 6667 50  0000 C CNN
+F 1 "S1B-13-F" H 3100 6576 50  0000 C CNN
+F 2 "Diode_SMD:D_SMA" H 3100 6450 50  0001 C CNN
 F 3 "~" H 3100 6450 50  0001 C CNN
 	1    3100 6450
@@
 	3650 6950 3700 6950
 $Comp
-L Device:D D?
+L Device:D D2
 U 1 1 607EA962
 P 4800 4750
-F 0 "D?" H 4800 4967 50  0000 C CNN
-F 1 "D" H 4800 4876 50  0000 C CNN
-F 2 "" H 4800 4750 50  0001 C CNN
+F 0 "D2" H 4800 4967 50  0000 C CNN
+F 1 "S1B-13-F" H 4800 4876 50  0000 C CNN
+F 2 "Diode_SMD:D_SMA" H 4800 4750 50  0001 C CNN
 F 3 "~" H 4800 4750 50  0001 C CNN
 	1    4800 4750
@@
 	6950 4400 6950 7800
 $Comp
-L Device:C C?
+L Device:C C6
 U 1 1 608C07ED
 P 3500 1900
-F 0 "C?" H 3615 1946 50  0000 L CNN
-F 1 "18pF/10V" H 3615 1855 50  0000 L CNN
-F 2 "" H 3538 1750 50  0001 C CNN
+F 0 "C6" H 3615 1946 50  0000 L CNN
+F 1 "18pF/20V" H 3615 1855 50  0000 L CNN
+F 2 "Capacitor_SMD:C_0805_2012Metric" H 3538 1750 50  0001 C CNN
 F 3 "~" H 3500 1900 50  0001 C CNN
 	1    3500 1900
@@
 $EndComp
 $Comp
-L Device:C C?
+L Device:C C4
 U 1 1 608C0CA6
 P 3250 2450
-F 0 "C?" H 3365 2496 50  0000 L CNN
-F 1 "18pF/10V" H 3365 2405 50  0000 L CNN
-F 2 "" H 3288 2300 50  0001 C CNN
+F 0 "C4" H 3365 2496 50  0000 L CNN
+F 1 "18pF/20V" H 3365 2405 50  0000 L CNN
+F 2 "Capacitor_SMD:C_0805_2012Metric" H 3288 2300 50  0001 C CNN
 F 3 "~" H 3250 2450 50  0001 C CNN
 	1    3250 2450
@@
 Wire Wire Line
 	5750 3350 6250 3350
+$Comp
+L CNC:NUP2114UCMR6T1G U1
+U 1 1 607223C1
+P 2100 1600
+F 0 "U1" H 2000 1000 50  0000 C CNN
+F 1 "NUP2114UCMR6T1G" H 2000 900 50  0000 C CNN
+F 2 "Package_TO_SOT_SMD:SOT-23-6" H 2100 1600 50  0001 C CNN
+F 3 "" H 2100 1600 50  0001 C CNN
+	1    2100 1600
+	1    0    0    -1
+$EndComp
+Text Label 1850 1500 0    50   ~ 0
+J2_D+
+Text Label 1850 1600 0    50   ~ 0
+J2_D-
 $EndSCHEMATC
