File: electronics/control/endstops.sch (KiCad schematic (older format))
At the start: 30 parts

Commit message: Add the PCB.
Parts:
- C16, C17, C18, C19, C20, C21: renamed from C?; value 0.1µF/10V -> 0.1µF/20V; footprint (none) -> Capacitor_SMD:C_0805_2012Metric
- J13, J14, J15, J16, J17, J18: renamed from J?; footprint (none) -> Connector_JST:JST_XH_B3B-XH-A_1x03_P2.50mm_Vertical
- R40, R41, R42, R43, R44, R45, R46, R47, R48, R49, R50, R51: renamed from R?; footprint (none) -> Resistor_SMD:R_0805_2012Metric
- RV4, RV5, RV6, RV7, RV8, RV9: renamed from RV?; footprint (none) -> Resistor_SMD:R_0805_2012Metric
Other:
- moved on the sheet: C16, C17, C20, C21, J13, J14, J17, J18, R40, R41, R42, R43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
