File: electronics/control/mcu.sch (KiCad schematic (older format))
At the start: 46 parts

Commit message: Add the PCB.
Parts:
- removed J?: RESET_ISP_BOOT, symbol Connector:Conn_01x03_Female
- removed J?: ETHERNET, symbol Connector_Generic:Conn_02x05_Odd_Even
- removed J? (x4): IO, symbol Connector:Conn_01x02_Female
- added C31, C32: 0.1µF/20V, Capacitor_SMD:C_0805_2012Metric, symbol Device:C
- added J34: ETHERNET, Connector_IDC:IDC-Header_2x06_P2.54mm_Vertical, symbol Connector_Generic:Conn_02x06_Odd_Even
- added R59: 1.5k, Resistor_SMD:R_0805_2012Metric, symbol Device:R
- C22, C28, C29, C30, C33: renamed from C?; value 0.1µF/10V -> 0.1µF/20V; footprint (none) -> Capacitor_SMD:C_0805_2012Metric
- C23: renamed from C?; value 1µF/10V -> 1µF/20V; footprint (none) -> Capacitor_SMD:C_0805_2012Metric
- C24, C25, C26: renamed from C?; footprint (none) -> Capacitor_SMD:C_0805_2012Metric
- C27: renamed from C?; value 10µF/10V Low ESR -> 10µF/20V; footprint (none) -> Capacitor_SMD:C_0805_2012Metric
- J19, J22: renamed from J?; footprint (none) -> Connector_JST:JST_XH_B4B-XH-A_1x04_P2.50mm_Vertical
- J21, J26, J28: renamed from J?; footprint (none) -> Connector_JST:JST_XH_B6B-XH-A_1x06_P2.50mm_Vertical
- J23: renamed from J?; footprint (none) -> Connector_IDC:IDC-Header_2x10_P2.54mm_Vertical
- J24, J29: renamed from J?; footprint (none) -> Connector_JST:JST_XH_B8B-XH-A_1x08_P2.50mm_Vertical
- J25: renamed from J?; footprint (none) -> Connector_JST:JST_XH_B7B-XH-A_1x07_P2.50mm_Vertical
- J33: renamed from J?; value SD_CARD -> MICROSD_CARD; footprint (none) -> Connector_Card:microSD_HC_Hirose_DM3D-SF
- L1: renamed from L?; footprint (none) -> Inductor_SMD:L_0805_2012Metric
- Q8: renamed from Q?; footprint (none) -> Package_TO_SOT_SMD:SOT-23
- R52, R53, R54, R55, R56, R57, R58, R60, R61, R62, R63, R64, R65, R66: renamed from R?; footprint (none) -> Resistor_SMD:R_0805_2012Metric
- SW1, SW2: renamed from SW?; footprint (none) -> Button_Switch_THT:SW_PUSH_6mm_H5mm
- Y1: renamed from Y?; footprint (none) -> Crystal:Crystal_SMD_Abracon_ABM3-2Pin_5.0x3.2mm
- gave numbers to parts that had none: 1
Connections:
- net +3V3: now also C31.2, C32.2, J34.2 (Pin_2)
- net ENET_CRS: now also J34.6 (Pin_6)
- net ENET_MDC: now also J34.11 (Pin_11)
- net ENET_MDIO: now also J34.12 (Pin_12)
- net ENET_REF_CLK: now also J34.10 (Pin_10)
- net ENET_RXD0: now also J34.7 (Pin_7)
- net ENET_RXD1: now also J34.8 (Pin_8)
- net ENET_RX_ER: now also J34.9 (Pin_9)
- net ENET_TXD0: now also J34.3 (Pin_3)
- net ENET_TXD1: now also J34.4 (Pin_4)
- net ENET_TX_EN: now also J34.5 (Pin_5)
- net GNDD: now also C31.1, C32.1, J34.1 (Pin_1)
- net P4_28: now also J24.8 (Pin_8)
- net P4_29: now also J24.7 (Pin_7)
- net USB_D+: now also R59.2; no longer Q8.3 (D)
- net Y_DIR: now also U14.48 (P0[10]); no longer U14.49 (P0[11])
- net Y_EN: now also U14.49 (P0[11]); no longer U14.48 (P0[10])
- net P1_30: no longer names the net of U14.21 (P1[30])
- net P1_31: no longer names the net of U14.20 (P1[31])
- net P2_12: no longer names the net of U14.51 (P2[12])
- net P2_13: no longer names the net of U14.50 (P2[13])
- net P3_25: no longer names the net of U14.27 (P3[25])
- net P3_26: no longer names the net of U14.26 (P3[26])
- net PO_21: no longer names the net of U14.57 (P0[21])
- net PO_21: no longer J24.8 (Pin_8)
- net PO_22: no longer names the net of U14.56 (P0[22])
- net PO_22: no longer J24.7 (Pin_7)
- new net: Q8.3 (D), R59.1
- no-connect marks 9 -> 17
Other:
- note added: "One per VDD"
- note added: "microSD Card"
- note removed: "One per VDD(3V3)"
- note removed: "SD Card"
- moved on the sheet: C33, Q8
