File: electronics/control/spindle.sch (KiCad schematic (older format))
At the start: 31 parts, among them U7 MOCD217R2M, U8 MOCD217R2M, U8 TS912

Commit message: Add the PCB.
Parts:
- removed C?: 100µF/50V, symbol Device:CP
- removed D?: D, symbol Device:D
- removed J?: MOTOR_POWER_12V_TO_30V, symbol Connector:Conn_01x02_Female
- removed Q?: Q_NMOS_DGS, symbol Device:Q_NMOS_DGS
- removed Q?: IRFS3006TRLPBF, symbol Device:Q_NMOS_GDS
- removed R?: 10k, symbol Device:R
- removed U?: MCP1416, Package_TO_SOT_SMD:SOT-23-5, symbol Driver_FET:MCP1416
- removed U?: MC7809, symbol CNC:MC7809
- added C15: 1µF/20V, Capacitor_SMD:C_0805_2012Metric, symbol Device:C
- added Q6: 2N7002-7-F, Package_TO_SOT_SMD:SOT-23, symbol Device:Q_NMOS_GSD
- C11: renamed from C?; value 10pF/10V -> 10pF/20V; footprint (none) -> Capacitor_SMD:C_0805_2012Metric
- C13: renamed from C?; value 47nF -> 47nF/20V; footprint (none) -> Capacitor_SMD:C_0805_2012Metric
- C14: renamed from C?; value 100nF -> 0.1µF/20V; footprint (none) -> Capacitor_SMD:C_0805_2012Metric
- D3: renamed from D?; value D -> S1B-13-F; footprint (none) -> Diode_SMD:D_SMA
- J10: renamed from J?; footprint (none) -> Connector_JST:JST_XH_B3B-XH-A_1x03_P2.50mm_Vertical
- J11: renamed from J?; footprint (none) -> Connector_JST:JST_XH_B2B-XH-A_1x02_P2.50mm_Vertical
- J12: renamed from J?; footprint (none) -> Connector_JST:JST_XH_B5B-XH-A_1x05_P2.50mm_Vertical
- JP11, JP12: renamed from JP?; footprint (none) -> Connector_PinHeader_2.54mm:PinHeader_1x03_P2.54mm_Vertical
- R30: renamed from R?; value 1k -> 50k; footprint (none) -> Resistor_SMD:R_0805_2012Metric
- R31, R32, R33, R34, R35, R36, R37, R39: renamed from R?; footprint (none) -> Resistor_SMD:R_0805_2012Metric
- RV2: renamed from RV?; footprint (none) -> Resistor_SMD:R_0805_2012Metric
- RV3: renamed from RV?; value R_POT -> POT_10k; footprint (none) -> Potentiometer_THT:Potentiometer_Bourns_3266Y_Vertical
- U7, U8: footprint (none) -> Package_SO:SOIC-8_3.9x4.9mm_P1.27mm
- U9: renamed from U8; footprint (none) -> Package_SO:SOIC-8_3.9x4.9mm_P1.27mm
Connections:
- net MOTOR_V+ is gone; now on an unnamed net: J11.1 (Pin_1)
- net CONTROLLER_10V: now also C15.1
- net CONTROLLER_EN: now also Q6.3 (D)
- net CONTROLLER_GND: now also D3.2 (A), C15.2, Q6.2 (S); no longer D3.1 (K)
- net at R33.1, U7.3: now also D3.1 (K); no longer D3.2 (A)
- net at R39.1: now also Q6.1 (G)
- net at U8.8: now also J11.2 (Pin_2)
- net MOTOR_GND: no longer names the net of U8.7
Other:
- note added: "DC MOTOR CONTROLLER"
- note added: "Hall Effect Sensor"
- note removed: "DC MOTOR CONTROLLER \nWS55-180/WS55-220"
- moved on the sheet: J11, J12, R36, R39, RV3, U8A, U9A, U9B, U9C
