File: electronics/teensy/control/control.sch (KiCad schematic (older format))
At the start: 0 parts

Commit message: Add gerber files
Connections:
- no-connect marks 1 -> 0
Changed lines of the file:
@@
 Wire Wire Line
 	1750 4600 1950 4600
-NoConn ~ 3500 3650
 $EndSCHEMATC
